File: src/RS485-Module/RS485-Module.kicad_pcb (KiCad board)
At the start: 2 copper layers, 62.7 x 33.8 mm, 29 parts, among them J1 Jumper_NO, J2 Jumper_NO, J3 Jumper_NO, J4 Jumper_NO, J5 Jumper_NO, J6 Jumper_NO, J7 Jumper_NO, J8 Jumper_NO, P1 5015680807, P2 282837-2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

Commit message: finished rev 1 routing
Parts:
- moved D1 25.6 mm to (173.6, 97.8)
- moved R1 22.4 mm to (167.4, 97.8)
- moved J6 16.6 mm to (173.9, 111.1)
- moved J2 15.8 mm to (173.8, 114.2)
- moved J1 11.2 mm to (173.9, 103.6)
- moved J3 8.69 mm to (173.9, 106.7)
- moved J4 7.67 mm to (173.9, 109.6)
- moved J7 4.72 mm to (173.9, 105.2)
- moved J8 2.85 mm to (173.8, 112.6)
- moved J5 2.72 mm to (173.9, 108.1)
- moved R6 2.67 mm to (166.2, 107.8)
- moved R2 2.29 mm to (161.8, 106.9)
- moved D2 2.22 mm to (169.8, 106.9)
- moved D3 1.63 mm to (169.9, 111.6)
- moved R5 1.52 mm to (161.8, 112.3)
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Routing:
- net Z: track 0.00 -> 40.1 mm, vias 0 -> 1
- net Y: track 0.00 -> 38.4 mm, vias 0 -> 1
- net B: track 0.00 -> 34.8 mm, vias 0 -> 1
- net Net-(J1-B): track 0.00 -> 32.1 mm
- net A: track 0.00 -> 30.2 mm
- net Net-(J5-B): track 0.00 -> 27.5 mm, vias 0 -> 2
- net Net-(J3-B): track 0.00 -> 25.9 mm
- net Net-(J7-B): track 0.00 -> 25.7 mm, vias 0 -> 2
- net MCU_TX: track 0.00 -> 22.7 mm
- net MCU_RX: track 0.00 -> 19.7 mm
- net Earth: track 0.00 -> 19.4 mm, vias 0 -> 8
- net 3.3V: track 0.00 -> 15.6 mm, vias 0 -> 6
- net Net-(D1-Pad1): track 0.00 -> 3.94 mm
- net Net-(U1-Z): track 0.00 -> 3.17 mm
- net Net-(U1-Y): track 0.00 -> 3.07 mm
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- added copper zone on In2.Cu, net 3.3V
- added copper zone on B.Cu, net Earth
- added copper zone on F.Cu, net Earth
- added copper zone on In1.Cu, net Earth
Other:
- copper layers 2 -> 4
- board text added: "A0009 RS485 Module"
- board text added: "Rev 1.0"
